File: HUSB238A PD Sink controller/HUSB238A PD Sink controller.kicad_pcb (KiCad board)
At the start: 2 copper layers, 50.8 x 50.8 mm, 114 parts, among them J1 VBUS, J2 VSET, J3 I2C, J4 ISET, Q1 CJAC70P06, U1 TPD4E05U06DQA, U2 HUSB238A

Commit message: Fix resistor values
Parts:
- R2: value 20kΩ -> 200kΩ
Changed lines of the file:
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@@
 			)
 		)
-		(property "Value" "20kΩ"
-			(at 0 1.43 0)
+		(property "Value" "200kΩ"
+			(at 3.556 0.0635 0)
 			(layer "F.Fab")
 			(effects
@@
 			)
 		)
-		(property "LCSC Part #" "C4184"
+		(property "LCSC Part #" "C25811"
 			(at 0 0 180)
 			(unlocked yes)
@@
 				(font
 					(size 0.001 0.001)
+					(thickness 0.15)
 				)
 			)
@@
 				(font
 					(size 0.001 0.001)
+					(thickness 0.15)
 				)
 			)
@@
 				(font
 					(size 0.001 0.001)
+					(thickness 0.15)
 				)
 			)
@@
 				(font
 					(size 0.001 0.001)
+					(thickness 0.15)
 				)
 			)
@@
 		(tags "resistor handsolder")
 		(property "Reference" "R8"
-			(at 2.895 0 -90)
+			(at 2.895 0 270)
 			(unlocked yes)
 			(layer "F.SilkS")
@@
 		(tags "resistor handsolder")
 		(property "Reference" "R9"
-			(at 2.895 0 -90)
+			(at 2.895 0 270)
 			(unlocked yes)
 			(layer "F.SilkS")
@@
 				(font
 					(size 0.001 0.001)
+					(thickness 0.15)
 				)
 			)
@@
 				(font
 					(size 0.001 0.001)
+					(thickness 0.15)
 				)
 			)
@@
 				(font
 					(size 0.001 0.001)
+					(thickness 0.15)
 				)
 			)
@@
 				(font
 					(size 0.001 0.001)
+					(thickness 0.15)
 				)
 			)
@@
 				(font
 					(size 0.001 0.001)
+					(thickness 0.15)
 				)
 			)
@@
 				(font
 					(size 0.001 0.001)
+					(thickness 0.15)
 				)
 			)
@@
 				(font
 					(size 0.001 0.001)
+					(thickness 0.15)
 				)
 			)
@@
 				(font
 					(size 0.001 0.001)
+					(thickness 0.15)
 				)
 			)
@@
 				(font
 					(size 0.001 0.001)
+					(thickness 0.15)
 				)
 			)
@@
 				(font
 					(size 0.001 0.001)
+					(thickness 0.15)
 				)
 			)
@@
 		)
 		(property "Value" "15V"
-			(at 0.1 1.9 180)
+			(at 3.175 0 180)
 			(layer "F.Fab")
 			(effects
@@
 				(font
 					(size 0.001 0.001)
+					(thickness 0.15)
 				)
 			)
@@
 				(font
 					(size 0.001 0.001)
+					(thickness 0.15)
 				)
 			)
@@
 				(font
 					(size 0.001 0.001)
+					(thickness 0.15)
 				)
 			)
@@
 				(font
 					(size 0.001 0.001)
+					(thickness 0.15)
 				)
 			)
@@
 				(font
 					(size 0.001 0.001)
+					(thickness 0.15)
 				)
 			)
@@
 				(font
 					(size 0.001 0.001)
+					(thickness 0.15)
 				)
 			)
@@
 		(tags "resistor handsolder")
 		(property "Reference" "R7"
-			(at 2.895 0 -90)
+			(at 2.895 0 270)
 			(unlocked yes)
 			(layer "F.SilkS")
@@
 				(font
 					(size 0.001 0.001)
+					(thickness 0.15)
 				)
 			)
@@
 				(font
 					(size 0.001 0.001)
+					(thickness 0.15)
 				)
 			)
@@
 		(tags "resistor handsolder")
 		(property "Reference" "R10"
-			(at 2.895 0 -90)
+			(at 2.895 0 270)
 			(unlocked yes)
 			(layer "F.SilkS")
@@
 				(font
 					(size 0.001 0.001)
+					(thickness 0.15)
 				)
 			)
@@
 				(font
 					(size 0.001 0.001)
+					(thickness 0.15)
 				)
 			)
@@
 				(font
 					(size 0.001 0.001)
+					(thickness 0.15)
 				)
 			)
@@
 				(font
 					(size 0.001 0.001)
+					(thickness 0.15)
 				)
 			)
@@
 				(font
 					(size 0.001 0.001)
+					(thickness 0.15)
 				)
 			)
@@
 				(font
 					(size 0.001 0.001)
+					(thickness 0.15)
 				)
 			)
@@
 		)
 		(property "Value" "TPD4E05U06DQA"
-			(at 0.01829 2.5 90)
+			(at 0.01829 7.874 180)
 			(layer "F.Fab")
 			(effects
@@
 				(font
 					(size 0.001 0.001)
+					(thickness 0.15)
 				)
 			)
@@
 				(font
 					(size 0.001 0.001)
+					(thickness 0.15)
 				)
 			)
@@
 				(font
 					(size 0.001 0.001)
+					(thickness 0.15)
 				)
 			)
@@
 				(font
 					(size 0.001 0.001)
+					(thickness 0.15)
 				)
 			)
@@
 				(font
 					(size 0.001 0.001)
+					(thickness 0.15)
 				)
 			)
@@
 				(font
 					(size 0.001 0.001)
+					(thickness 0.15)
 				)
 			)
@@
 		)
 		(property "Value" "≥48V TVS Clamp"
-			(at 0 2.1 0)
+			(at -0.3175 1.778 0)
 			(layer "F.Fab")
 			(effects
@@
 		)
 		(property "Value" "100kΩ"
-			(at 0 1.43 0)
+			(at 4.064 0 0)
 			(layer "F.Fab")
 			(effects
