File: HUSB238A PD Sink controller/HUSB238A PD Sink controller.kicad_sch (KiCad schematic)
At the start: 29 parts, among them J1 VBUS, J2 VSET, J3 I2C, J4 ISET, Q1 CJAC70P06, U1 TPD4E05U06DQA, U2 HUSB238A

Commit message: diodes
Parts:
- D2: symbol Device:D_Schottky_Small -> Device:D_Zener_Small
Changed lines of the file:
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@@
 	)
 	(symbol
-		(lib_id "Device:D_Schottky_Small")
+		(lib_id "Device:D_Zener_Small")
 		(at 208.28 39.37 90)
 		(mirror x)
@@
 		)
 		(property "Value" "15V"
-			(at 205.994 41.148 90)
+			(at 206.502 41.148 90)
 			(effects
 				(font
